File: Board/RGBPS Breakout/RGBPS Breakout.kicad_sch (KiCad schematic)
At the start: 12 parts, among them IC1 APDS-9999, J1 Conn_01x04_Pin, J2 Conn_01x01_Pin

Commit message: routing
Parts:
- D1: value 3.2V WHITE -> 2.8V WHITE
- IC1: footprint (none) -> APDS-9999:APDS9999; Height 0.75 -> 0.8; Mouser Part Number (none) -> 630-APDS-9999; Mouser Price/Stock (none) -> https://www.mouser.co.uk/ProductDetail/Broadcom-Avago/APDS-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
- R1: value 1.667 -> 7.7
Connections:
- net +3.3V: now also D1.2 (A); no longer D1.1 (K)
- net at R1.1: now also D1.1 (K); no longer D1.2 (A)
Other:
- note added: "0.182W"
- moved on the sheet: D1
Changed lines of the file:
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@@
+		)
+	)
+	(text "0.182W"
+		(exclude_from_sim no)
+		(at 186.69 102.87 0)
+		(effects
+			(font
+				(size 0.762 0.762)
+			)
 		)
 	)
@@
 			)
 		)
-		(property "Value" "1.667"
+		(property "Value" "7.7"
 			(at 186.69 96.52 90)
 			(effects
@@
 	(symbol
 		(lib_id "Device:LED")
-		(at 175.26 100.33 0)
+		(at 175.26 100.33 180)
 		(unit 1)
 		(exclude_from_sim no)
@@
 		(fields_autoplaced yes)
 		(property "Reference" "D1"
-			(at 173.6725 93.98 0)
-			(effects
-				(font
-					(size 1.27 1.27)
-				)
-			)
-		)
-		(property "Value" "3.2V WHITE"
-			(at 173.6725 96.52 0)
+			(at 176.8475 92.71 0)
+			(effects
+				(font
+					(size 1.27 1.27)
+				)
+			)
+		)
+		(property "Value" "2.8V WHITE"
+			(at 176.8475 95.25 0)
 			(effects
 				(font
@@
 	(symbol
 		(lib_id "APDS-9999:APDS-9999")
-		(at 72.39 100.33 0)
-		(unit 1)
-		(exclude_from_sim no)
-		(in_bom yes)
-		(on_board yes)
-		(dnp no)
-		(fields_autoplaced yes)
+		(at 102.87 100.33 0)
+		(mirror y)
+		(unit 1)
+		(exclude_from_sim no)
+		(in_bom yes)
+		(on_board yes)
+		(dnp no)
 		(property "Reference" "IC1"
-			(at 87.63 92.71 0)
+			(at 87.884 96.266 0)
 			(effects
 				(font
@@
 		)
 		(property "Value" "APDS-9999"
-			(at 87.63 95.25 0)
-			(effects
-				(font
-					(size 1.27 1.27)
-				)
-			)
-		)
-		(property "Footprint" ""
-			(at 99.06 195.25 0)
+			(at 87.884 94.234 0)
+			(effects
+				(font
+					(size 1.27 1.27)
+				)
+			)
+		)
+		(property "Footprint" "APDS-9999:APDS9999"
+			(at 76.2 195.25 0)
 			(effects
 				(font
@@
 		)
 		(property "Datasheet" "https://docs.broadcom.com/doc/APDS-9999-DS"
-			(at 99.06 295.25 0)
+			(at 76.2 295.25 0)
 			(effects
 				(font
@@
 			)
 		)
-		(property "Description" "Ambient Light Sensors Integrated Digital RGB+PS"
-			(at 72.644 92.202 0)
-			(effects
-				(font
-					(size 1.27 1.27)
-				)
-				(hide yes)
-			)
-		)
-		(property "Height" "0.75"
-			(at 99.06 495.25 0)
+		(property "Description" "Optical Sensor Ambient 470nm, 550nm, 610nm I2C 6-SMD Module"
+			(at 102.616 92.202 0)
+			(effects
+				(font
+					(size 1.27 1.27)
+				)
+				(hide yes)
+			)
+		)
+		(property "Height" "0.8"
+			(at 76.2 495.25 0)
 			(effects
 				(font
@@
 			)
 		)
-		(property "Mouser Part Number" ""
-			(at 99.06 595.25 0)
+		(property "Mouser Part Number" "630-APDS-9999"
+			(at 76.2 595.25 0)
 			(effects
 				(font
@@
 			)
 		)
-		(property "Mouser Price/Stock" ""
-			(at 99.06 695.25 0)
+		(property "Mouser Price/Stock" "https://www.mouser.co.uk/ProductDetail/Broadcom-Avago/APDS-9999?qs=Cb2nCFKsA8qjJaAGveOY%252Bg%3D%3D"
+			(at 76.2 695.25 0)
 			(effects
 				(font
@@
 		)
 		(property "Manufacturer_Name" "Avago Technologies"
-			(at 99.06 795.25 0)
+			(at 76.2 795.25 0)
 			(effects
 				(font
@@
 		)
 		(property "Manufacturer_Part_Number" "APDS-9999"
-			(at 99.06 895.25 0)
-			(effects
-				(font
+			(at 76.2 895.25 0)
+			(effects
+				(font
+					(size 1.27 1.27)
+				)
+				(justify left top)
+				(hide yes)
+			)
+		)
+		(property "Arrow Part Number" ""
+			(at 76.2 995.25 0)
+			(effects
+				(font
+					(size 1.27 1.27)
+				)
+				(justify left top)
+				(hide yes)
+			)
+		)
+		(property "Arrow Price/Stock" ""
+			(at 76.2 1095.25 0)
+			(effects
+				(font
